Commit message: finished marble_husky_sensor_config_6

File: submitted_models/marble_husky_sensor_config_6/urdf/robot_from_sdf.xacro (robot description, xacro)
@@ -1,5 +1,5 @@
 <?xml version='1.0' encoding='utf-8'?>
-<robot name='marble_husky_sensor_config_1' xmlns:xacro='http://ros.org/wiki/xacro'>
-  <xacro:arg name="name" default="marble_husky_sensor_config_1"/>
+<robot name='marble_husky_sensor_config_6' xmlns:xacro='http://ros.org/wiki/xacro'>
+  <xacro:arg name="name" default="marble_husky_sensor_config_6"/>
   <xacro:property name="robot_namespace" value="$(arg name)"/>
   <link name='${robot_namespace}/base_link'>
@@ -72,5 +72,5 @@
       <origin xyz='0 0 0' rpy='0 -0 0'/>
       <geometry>
-        <mesh filename='package://marble_husky_sensor_config_1/meshes/base_link.dae' scale='1 1 1'/>
+        <mesh filename='package://marble_husky_sensor_config_6/meshes/base_link.dae' scale='1 1 1'/>
       </geometry>
     </visual>
@@ -78,5 +78,5 @@
       <origin xyz='0.478 0 0.26' rpy='0 0.5236 0'/>
       <geometry>
-        <mesh filename='package://marble_husky_sensor_config_1/meshes/realsense.dae' scale='1 1 1'/>
+        <mesh filename='package://marble_husky_sensor_config_6/meshes/realsense.dae' scale='1 1 1'/>
       </geometry>
     </visual>
@@ -84,5 +84,5 @@
       <origin xyz='0.478 0 0.285' rpy='0 -0 0'/>
       <geometry>
-        <mesh filename='package://marble_husky_sensor_config_1/meshes/realsense.dae' scale='1 1 1'/>
+        <mesh filename='package://marble_husky_sensor_config_6/meshes/realsense.dae' scale='1 1 1'/>
       </geometry>
     </visual>
@@ -90,5 +90,5 @@
       <origin xyz='0.48 0 0.091' rpy='0 -0 0'/>
       <geometry>
-        <mesh filename='package://marble_husky_sensor_config_1/meshes/bumper.dae' scale='1 1 1'/>
+        <mesh filename='package://marble_husky_sensor_config_6/meshes/bumper.dae' scale='1 1 1'/>
       </geometry>
     </visual>
@@ -96,5 +96,5 @@
       <origin xyz='-0.48 0 0.091' rpy='0 -0 3.14159'/>
       <geometry>
-        <mesh filename='package://marble_husky_sensor_config_1/meshes/bumper.dae' scale='1 1 1'/>
+        <mesh filename='package://marble_husky_sensor_config_6/meshes/bumper.dae' scale='1 1 1'/>
       </geometry>
     </visual>
@@ -102,5 +102,5 @@
       <origin xyz='0 0 0' rpy='0 -0 0'/>
       <geometry>
-        <mesh filename='package://marble_husky_sensor_config_1/meshes/top_chassis.dae' scale='1 1 1'/>
+        <mesh filename='package://marble_husky_sensor_config_6/meshes/top_chassis.dae' scale='1 1 1'/>
       </geometry>
     </visual>
@@ -108,5 +108,5 @@
       <origin xyz='0.424 0 0.327' rpy='0 -0 0'/>
       <geometry>
-        <mesh filename='package://marble_husky_sensor_config_1/meshes/VLP16_base_1.dae' scale='1 1 1'/>
+        <mesh filename='package://marble_husky_sensor_config_6/meshes/VLP16_base_1.dae' scale='1 1 1'/>
       </geometry>
     </visual>
@@ -114,5 +114,5 @@
       <origin xyz='0.424 0 0.327' rpy='0 -0 0'/>
       <geometry>
-        <mesh filename='package://marble_husky_sensor_config_1/meshes/VLP16_base_2.dae' scale='1 1 1'/>
+        <mesh filename='package://marble_husky_sensor_config_6/meshes/VLP16_base_2.dae' scale='1 1 1'/>
       </geometry>
     </visual>
@@ -120,5 +120,5 @@
       <origin xyz='0.424 0 0.327' rpy='0 -0 0'/>
       <geometry>
-        <mesh filename='package://marble_husky_sensor_config_1/meshes/VLP16_scan.dae' scale='1 1 1'/>
+        <mesh filename='package://marble_husky_sensor_config_6/meshes/VLP16_scan.dae' scale='1 1 1'/>
       </geometry>
     </visual>
@@ -126,5 +126,5 @@
       <origin xyz='0.272 0 0.245' rpy='0 -0 0'/>
       <geometry>
-        <mesh filename='package://marble_husky_sensor_config_1/meshes/user_rail.dae' scale='1 1 1'/>
+        <mesh filename='package://marble_husky_sensor_config_6/meshes/user_rail.dae' scale='1 1 1'/>
       </geometry>
     </visual>
@@ -195,5 +195,5 @@
       <origin xyz='0 0 0' rpy='0 -0 0'/>
       <geometry>
-        <mesh filename='package://marble_husky_sensor_config_1/meshes/wheel.dae' scale='1 1 1'/>
+        <mesh filename='package://marble_husky_sensor_config_6/meshes/wheel.dae' scale='1 1 1'/>
       </geometry>
     </visual>
@@ -214,5 +214,5 @@
       <origin xyz='0 0 0' rpy='0 -0 0'/>
       <geometry>
-        <mesh filename='package://marble_husky_sensor_config_1/meshes/wheel.dae' scale='1 1 1'/>
+        <mesh filename='package://marble_husky_sensor_config_6/meshes/wheel.dae' scale='1 1 1'/>
       </geometry>
     </visual>
@@ -233,5 +233,5 @@
       <origin xyz='0 0 0' rpy='0 -0 0'/>
       <geometry>
-        <mesh filename='package://marble_husky_sensor_config_1/meshes/wheel.dae' scale='1 1 1'/>
+        <mesh filename='package://marble_husky_sensor_config_6/meshes/wheel.dae' scale='1 1 1'/>
       </geometry>
     </visual>
@@ -252,5 +252,5 @@
       <origin xyz='0 0 0' rpy='0 -0 0'/>
       <geometry>
-        <mesh filename='package://marble_husky_sensor_config_1/meshes/wheel.dae' scale='1 1 1'/>
+        <mesh filename='package://marble_husky_sensor_config_6/meshes/wheel.dae' scale='1 1 1'/>
       </geometry>
     </visual>
@@ -296,5 +296,5 @@
       <origin xyz='0 0 0.03' rpy='0 -0 0'/>
       <geometry>
-        <mesh filename='package://marble_husky_sensor_config_1/meshes/realsense.dae' scale='1 1 1'/>
+        <mesh filename='package://marble_husky_sensor_config_6/meshes/realsense.dae' scale='1 1 1'/>
       </geometry>
     </visual>
